File: APM_BLE.brd (EAGLE design)
At the start: 26.7 x 47.2 mm, 33 parts, among them J1 CON_HEADER_PRG_AVR_ICSP-PTH, J2 B2B-PH-K-S(LF)(SN), Q1 8MHz, Q2 PMV48XP, Q3 PMV48XP, U1 ATMEGA328P, U3 JDY-08

Commit message: Update battery voltage sense resistor values
Update battery voltage sense resistor values
Parts:
- R4: value TBD -> 200k 1%
- R5: value TBD -> 100k 1%
Changed lines of the file:
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@@
 <attribute name="VALUE" x="23.268" y="28.67" size="0.6096" layer="27" font="vector" ratio="20" rot="R270"/>
 </element>
-<element name="R4" library="SparkFun" package="0603-RES" value="TBD" x="24.9" y="15.1" smashed="yes" rot="R90">
+<element name="R4" library="SparkFun" package="0603-RES" value="200k 1%" x="24.9" y="15.1" smashed="yes" rot="R90">
 <attribute name="NAME" x="24.511" y="12.562" size="0.8128" layer="25" font="vector"/>
 <attribute name="VALUE" x="26.043" y="14.084" size="0.4064" layer="27" font="vector" rot="R90"/>
 </element>
-<element name="R5" library="SparkFun" package="0603-RES" value="TBD" x="25.1" y="8.8" smashed="yes" rot="R90">
+<element name="R5" library="SparkFun" package="0603-RES" value="100k 1%" x="25.1" y="8.8" smashed="yes" rot="R90">
 <attribute name="NAME" x="24.238" y="7.411" size="0.8128" layer="25" font="vector" rot="R90"/>
 <attribute name="VALUE" x="26.243" y="7.784" size="0.4064" layer="27" font="vector" rot="R90"/>
