File: APM_BLE.sch (EAGLE design)
At the start: 33 parts, among them J1 CON_HEADER_PRG_AVR_ICSP-PTH, J2 B2B-PH-K-S(LF)(SN), Q1 8MHz, Q2 PMV48XP, Q3 PMV48XP, U1 ATMEGA328P, U3 JDY-08

Commit message: Update battery voltage sense resistor values
Update battery voltage sense resistor values
Parts:
- R4: value TBD -> 200k 1%
- R5: value TBD -> 100k 1%
Changed lines of the file:
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@@
 <part name="J3" library="SparkFun-Connectors" deviceset="CONN_04" device=""/>
 <part name="GND13" library="SparkFun" deviceset="GND" device=""/>
-<part name="R4" library="SparkFun" deviceset="RESISTOR" device="0603-RES" value="TBD"/>
-<part name="R5" library="SparkFun" deviceset="RESISTOR" device="0603-RES" value="TBD"/>
+<part name="R4" library="SparkFun" deviceset="RESISTOR" device="0603-RES" value="200k 1%"/>
+<part name="R5" library="SparkFun" deviceset="RESISTOR" device="0603-RES" value="100k 1%"/>
 <part name="GND14" library="SparkFun" deviceset="GND" device=""/>
 <part name="C6" library="SparkFun" deviceset="CAP" device="0603-CAP" value="1nF"/>
