File: CADA/APM_BLE.brd (EAGLE design)
At the start: 26.7 x 47.2 mm, 33 parts, among them J1 CON_HEADER_PRG_AVR_ICSP-PTH, J2 B2B-PH-K-S(LF)(SN), Q1 8MHz, Q2 PMV48XP, Q3 PMV48XP, U1 ATMEGA328P, U3 JDY-08

Commit message: Latest files
Parts:
- R7: value 2k -> 100k
Changed lines of the file:
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@@
 <attribute name="VALUE" x="8.847" y="43.702" size="1.27" layer="27" rot="R180"/>
 </element>
-<element name="R7" library="SparkFun" package="0603-RES" value="2k" x="9.271" y="43.307" smashed="yes">
+<element name="R7" library="SparkFun" package="0603-RES" value="100k" x="9.271" y="43.307" smashed="yes">
 <attribute name="NAME" x="6.082" y="43.069" size="0.8128" layer="25" font="vector"/>
 <attribute name="VALUE" x="8.255" y="42.164" size="0.4064" layer="27" font="vector"/>
