File: CADA/APM_BLE.sch (EAGLE design)
At the start: 33 parts, among them J1 CON_HEADER_PRG_AVR_ICSP-PTH, J2 B2B-PH-K-S(LF)(SN), Q1 8MHz, Q2 PMV48XP, Q3 PMV48XP, U1 ATMEGA328P, U3 JDY-08

Commit message: Latest files
Parts:
- R7: value 2k -> 100k
Changed lines of the file:
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@@
 <part name="JP3" library="BC9VPC_ShortenedSilkScreen" deviceset="M04" device="PTH"/>
 <part name="D1" library="diode" deviceset="MBR0520LT" device=""/>
-<part name="R7" library="SparkFun" deviceset="RESISTOR" device="0603-RES" value="2k"/>
+<part name="R7" library="SparkFun" deviceset="RESISTOR" device="0603-RES" value="100k"/>
 <part name="GND6" library="SparkFun" deviceset="GND" device=""/>
 <part name="LOGO1" library="ohw-logo" deviceset="OSHW_LOGO_FILL" device="X0200-NT"/>
