File: CAD_A/APM_BLE.sch (EAGLE design)
At the start: 33 parts, among them J1 CON_HEADER_PRG_AVR_ICSP-PTH, J2 B2B-PH-K-S(LF)(SN), Q1 8MHz, Q2 PMV48XP, Q3 PMV48XP, U1 ATMEGA328P, U3 JDY-08

Commit message: Minor updates
Minor Updates
Parts:
- R4: value 200k 1% -> 200k, 1%
- R5: value 100k 1% -> 100k, 1%
Changed lines of the file:
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@@
 <part name="J3" library="SparkFun-Connectors" deviceset="CONN_04" device=""/>
 <part name="GND13" library="SparkFun" deviceset="GND" device=""/>
-<part name="R4" library="SparkFun" deviceset="RESISTOR" device="0603-RES" value="200k 1%"/>
-<part name="R5" library="SparkFun" deviceset="RESISTOR" device="0603-RES" value="100k 1%"/>
+<part name="R4" library="SparkFun" deviceset="RESISTOR" device="0603-RES" value="200k, 1%"/>
+<part name="R5" library="SparkFun" deviceset="RESISTOR" device="0603-RES" value="100k, 1%"/>
 <part name="GND14" library="SparkFun" deviceset="GND" device=""/>
 <part name="C6" library="SparkFun" deviceset="CAP" device="0603-CAP" value="1nF"/>

Commit message: unknown changes
Changed lines of the file:
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@@
 </instance>
 <instance part="U3" gate="G$1" x="109.22" y="43.18"/>
-<instance part="S2" gate="G$1" x="127" y="147.32" rot="R90"/>
+<instance part="S2" gate="G$1" x="127" y="147.32" smashed="yes" rot="R90">
+<attribute name="NAME" x="124.46" y="144.78" size="1.778" layer="95" rot="R90"/>
+<attribute name="VALUE" x="129.54" y="144.78" size="1.778" layer="96" rot="R90" display="off"/>
+</instance>
 <instance part="F1" gate="G$1" x="38.1" y="160.02"/>
 <instance part="SUPPLY1" gate="G$1" x="30.48" y="167.64"/>
