File: CAD_B/APM_BLE.sch (EAGLE design)
At the start: 33 parts, among them J1 CON_HEADER_PRG_AVR_ICSP-PTH, J2 B2B-PH-K-S(LF)(SN), Q1 8MHz, Q2 PMV48XP, Q3 PMV48XP, U1 ATMEGA328P, U3 JDY-08

Commit message: pnums added and cap change
Changed 10uF cap to 0603, updated PCB
added farnell pnums
Parts:
- removed C5: 10uF, rcl:C-EUC0805K
- added C7: 10uF, SparkFun:CAP0603-CAP
- C1, C10, C2, C3, C4, C6, D1, D3, F1, FID1, FID2, J1, JP1, LOGO1, R1, R3, R6, S2, U3: OC_FARNELL (none) -> unknown
- J2: value B2B-PH-K-S(LF)(SN) -> S2B-PH-SM4-TB(LF)(SN); MF (none) -> JST (JAPAN SOLDERLESS TERMINALS); MPN (none) -> S2B-PH-SM4-TB(LF)(SN); OC_FARNELL (none) -> 9492615
- J3, JP3: value (none) -> 1X4 PIN HEADER; OC_FARNELL (none) -> unknown
- J4, JP2: value (none) -> NO_FIT; OC_FARNELL (none) -> unknown
- Q1: value 8MHz -> 8MHz CSTCE8M00G55-R0; MF (none) -> MURATA; MPN (none) -> CSTCE8M00G55-R0; OC_FARNELL (none) -> 2443270
- Q2, Q3: value PMV48XP -> PMV48XP or DMP2035U; MF (none) -> DIODES INC.; MPN (none) -> DMP2035U; OC_FARNELL (none) -> 2061419
- R2: value 10K -> 10K, 1%; OC_FARNELL (none) -> unknown
- R4: value 200k 1% -> 200k, 1%; OC_FARNELL (none) -> unknown
- R5: value 100k 1% -> 100k, 1%; OC_FARNELL (none) -> unknown
- R7: value 100k -> 100k, 1%; OC_FARNELL (none) -> unknown
- U1: MF (none) -> MICROCHIP; MPN (none) -> ATMEGA328P-AU; OC_FARNELL (none) -> 1715486
Connections:
- net N$4 renamed FS_D
- net +3V3: now also C7.2; no longer C5.1
- net GND: now also C7.1; no longer C5.2
Other:
- note added: "CONSIDER 3 PIN JST BATTERY HOLDER WITH SAFETY SCREW AND JST CONNECTOR 2489CN"
- note added: "SPI CSS BREAKOUT"
- note added: "USE ONLY NON_RECHARGABLE BATTERIES. APPROX 3V0 INPUT."
- note removed: "SETUP FOR NON_RECHARGABLE BATTERIES. APPROX 3V0 INPUT."
- note removed: "TO 2 X AAA OR AA BATTERY HOLDER EG FROM KITRONIC"
- moved on the sheet: JP3

Commit message: Minor updates
Minor Updates
Parts:
- added C11, C9: 22pF, SparkFun:CAP0603-CAP
- added C5: 0.1uF, SparkFun:CAP0603-CAP
- added C8: 10uF, SparkFun:CAP0603-CAP
- added Q4: 8MHz, adafruit:CRYSTALHC49UP
- added Q5: (no value), crystal:CRYSTALCTS406
- added R8, R9: 0R0, SparkFun:RESISTOR0603-RES
- added S1: MOMENTARY-SWITCH-SPST-SMD-6.0X3.5MM, SparkFun-Switches:MOMENTARY-SWITCH-SPST-SMD-6.0X3.5MM
- added U2: TSYS01, TSYS01:TSYS01
- F1: value MF-MSMF050-2 500mA -> MSMF110-2, 1.1A; MF (none) -> BOURNS; MPN (none) -> MF-MSMF110-2; OC_FARNELL unknown -> 9350330
- Q1: value 8MHz CSTCE8M00G55-R0 -> 8MHz CSTCE8M00G55-R0
- R4: value 200k, 1% -> 390k, 1%
- U3: device JDY-08:JDY-08 -> JDY-08:JDY-08JDY-08_MODULE
Connections:
- removed net A4: JP3.4, R1.1, U1.PC4(ADC4/SDA)
- removed net A5: JP3.3, R3.1, U1.PC5(ADC5/SCL)
- new net A4_SDA: JP3.4, R1.1, U1.PC4(ADC4/SDA), U2.SDI/SDA
- new net A5_SCL: JP3.3, R3.1, U1.PC5(ADC5/SCL), U2.SCLK/SCL
- new net N$10: R8.1, U2.PS
- new net N$4: R9.1, U2.CSB
- new net N$6: U2.INT, U2.INT/EXT
- net +3V3: now also C5.2, C8.2, R8.2, R9.2, U2.VDD
- net GND: now also C5.1, C8.1, U2.EXP, U2.VSS
Other:
- note added: "6-9, 12-14 NC"
- note added: "I2C HEADER PINOUT = EBAY SHT31, BME280 SOME ADAFRUIT"
- note added: "NC"
- note added: "ROUTE AROUND FOR THERMAL BARRIER"
- moved on the sheet: C4, JP2, Q3

Commit message: unknown changes
Other:
- note added: "FET NOT TURNING ON FULLY CHANGE TO ANOTHER PART!"
Changed lines of the file:
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@@
 <text x="162.56" y="35.56" size="1.778" layer="91">6-9, 12-14 NC</text>
 <text x="162.56" y="33.02" size="1.778" layer="91">ROUTE AROUND FOR THERMAL BARRIER</text>
+<text x="-17.78" y="38.1" size="1.778" layer="91">FET NOT TURNING ON FULLY CHANGE TO ANOTHER PART!</text>
 </plain>
 <instances>
